File: Hardware/SparkFun_Cryptographic_Co-processor_ATECC608A.brd (EAGLE design)
At the start: 25.4 x 25.4 mm, 41 parts, among them J1 QWIIC, J2 QWIIC, J3 PTH, U1 ATECC608A

Commit message: eng 1st run checklist stuff
-added qwiic logo as device so it has logo in SCH
-update vector font to "non-legacy"
-cleaned up assembly sheet view attribute placement
-IC datasheet (summary only)
-measures updated, PNG and PDF files created.
-Exported SCH as PDF in docs
Parts:
- LOGO3: value (none) -> QWIIC_LOGO_4MM
- renumbered U$16 to LOGO3
Other:
- board text added: "UNITS: INCHES"
Changed lines of the file:
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@@
 <layer number="27" name="tValues" color="7" fill="1" visible="no" active="yes"/>
 <layer number="28" name="bValues" color="7" fill="1" visible="no" active="yes"/>
-<layer number="29" name="tStop" color="7" fill="3" visible="yes" active="yes"/>
+<layer number="29" name="tStop" color="7" fill="3" visible="no" active="yes"/>
 <layer number="30" name="bStop" color="7" fill="6" visible="no" active="yes"/>
-<layer number="31" name="tCream" color="7" fill="4" visible="yes" active="yes"/>
+<layer number="31" name="tCream" color="7" fill="4" visible="no" active="yes"/>
 <layer number="32" name="bCream" color="7" fill="5" visible="no" active="yes"/>
 <layer number="33" name="tFinish" color="6" fill="3" visible="no" active="yes"/>
@@
 <text x="24.3586" y="12.8524" size="1.27" layer="16" font="vector" ratio="24" rot="SMR270" align="center">v10</text>
 <text x="16.51" y="-12.7" size="1.778" layer="51" font="vector">Pete Lewis</text>
-<dimension x1="0" y1="0" x2="0" y2="25.4" x3="-15.24" y3="12.7" textsize="1.016" layer="47" unit="inch" visible="yes"/>
-<dimension x1="2.54" y1="22.86" x2="2.54" y2="0" x3="-11.43" y3="11.43" textsize="1.016" layer="47" unit="inch" visible="yes"/>
-<dimension x1="2.54" y1="22.86" x2="0" y2="22.86" x3="1.27" y3="26.67" textsize="1.016" layer="47" unit="inch" visible="yes"/>
-<dimension x1="22.86" y1="22.86" x2="0" y2="22.86" x3="11.43" y3="30.48" textsize="1.016" layer="47" unit="inch" visible="yes"/>
-<dimension x1="22.86" y1="2.54" x2="22.86" y2="0" x3="29.21" y3="1.27" textsize="1.016" layer="47" unit="inch" visible="yes"/>
+<dimension x1="0" y1="0" x2="0" y2="25.4" x3="-15.24" y3="12.7" textsize="1.27" layer="47" unit="inch"/>
+<dimension x1="2.54" y1="22.86" x2="2.54" y2="0" x3="-11.43" y3="11.43" textsize="1.27" layer="47" unit="inch"/>
+<dimension x1="2.54" y1="22.86" x2="0" y2="22.86" x3="1.27" y3="26.67" textsize="1.27" layer="47" unit="inch"/>
+<dimension x1="22.86" y1="22.86" x2="0" y2="22.86" x3="11.43" y3="30.48" textsize="1.27" layer="47" unit="inch"/>
+<dimension x1="22.86" y1="2.54" x2="22.86" y2="0" x3="29.21" y3="1.27" textsize="1.27" layer="47" unit="inch"/>
 <rectangle x1="11.049" y1="11.7602" x2="11.4046" y2="11.7856" layer="41"/>
-<dimension x1="2.54" y1="2.54" x2="2.54" y2="0" x3="-3.81" y3="1.27" textsize="1.016" layer="47" unit="inch" visible="yes"/>
-<dimension x1="0" y1="25.4" x2="25.4" y2="25.4" x3="12.7" y3="34.29" textsize="1.016" layer="47" unit="inch" visible="yes"/>
-<dimension x1="22.86" y1="22.86" x2="22.86" y2="0" x3="36.83" y3="11.43" textsize="1.016" layer="47" unit="inch" visible="yes"/>
-<dimension x1="25.4" y1="0" x2="25.4" y2="25.4" x3="40.64" y3="12.7" textsize="1.016" layer="47" unit="inch" visible="yes"/>
-<dimension x1="0" y1="0" x2="0" y2="12.7" x3="-7.62" y3="6.35" textsize="1.016" textratio="15" layer="47" unit="inch" visible="yes"/>
-<dimension x1="25.4" y1="0" x2="25.4" y2="12.7" x3="33.02" y3="6.35" textsize="1.016" textratio="15" layer="47" unit="inch" visible="yes"/>
+<dimension x1="2.54" y1="2.54" x2="2.54" y2="0" x3="-3.81" y3="1.27" textsize="1.27" layer="47" unit="inch"/>
+<dimension x1="0" y1="25.4" x2="25.4" y2="25.4" x3="12.7" y3="34.29" textsize="1.27" layer="47" unit="inch"/>
+<dimension x1="22.86" y1="22.86" x2="22.86" y2="0" x3="36.83" y3="11.43" textsize="1.27" layer="47" unit="inch"/>
+<dimension x1="25.4" y1="0" x2="25.4" y2="25.4" x3="40.64" y3="12.7" textsize="1.27" layer="47" unit="inch"/>
+<dimension x1="0" y1="0" x2="0" y2="12.7" x3="-7.62" y3="6.35" textsize="1.27" textratio="15" layer="47" unit="inch"/>
+<dimension x1="25.4" y1="0" x2="25.4" y2="12.7" x3="33.02" y3="6.35" textsize="1.27" textratio="15" layer="47" unit="inch"/>
+<text x="12.7" y="-3.81" size="1.27" layer="47" font="vector" ratio="15" align="bottom-center">UNITS: INCHES</text>
 </plain>
 <attributes>
@@
 <attribute name="VALUE" x="12.7" y="16.002" size="0.6096" layer="27" font="vector" ratio="20" rot="R180" align="top-center"/>
 </element>
-<element name="U$16" library="SparkFun-Aesthetics" package="QWIIC_4MM" value="" x="22.733" y="17.0942" smashed="yes"/>
 <element name="D1" library="SparkFun-LED" package="LED-0603" value="RED" x="22.5806" y="7.62" smashed="yes">
 <attribute name="NAME" x="22.5806" y="8.255" size="0.6096" layer="25" font="vector" ratio="20" align="bottom-center"/>
 <attribute name="PROD_ID" value="DIO-00819" x="22.5806" y="7.62" size="1.778" layer="27" font="vector" ratio="15" display="off"/>
-<attribute name="VALUE" x="22.5806" y="6.985" size="0.6096" layer="27" font="vector" ratio="20" align="top-center"/>
+<attribute name="VALUE" x="22.6314" y="8.255" size="0.6096" layer="27" font="vector" ratio="20" rot="R180" align="top-center"/>
 </element>
 <element name="R3" library="SparkFun-Resistors" package="0603" value="1k" x="19.05" y="7.62" smashed="yes" rot="R180">
@@
 <element name="U$8" library="SparkFun-Aesthetics" package="CRYPTO_COPROCESSOR_LOGO_LARGE" value="" x="12.7" y="13.97" smashed="yes" rot="MR0"/>
 <element name="U$10" library="SparkFun-Aesthetics" package="CRYPTO_COPROCESSOR_LOGO_SMALL" value="" x="5.207" y="7.112" smashed="yes"/>
+<element name="LOGO3" library="SparkFun-Aesthetics" package="QWIIC_4MM" value="QWIIC_LOGO_4MM" x="22.733" y="17.0942" smashed="yes"/>
 </elements>
 <signals>
